File: grupo-1/Julio/amplificador/amplificador.kicad_pcb (KiCad board)
At the start: 2 copper layers, 40 x 25 mm, 0 parts

Commit message: avance bryan, actividad 1 fin
Parts:
- added C1: C_Polarized, Capacitor_THT:CP_Radial_D8.0mm_P3.50mm, F.Cu at (183.0, 106.0)
- added C2: C_Polarized, Capacitor_THT:CP_Radial_D8.0mm_P3.50mm, F.Cu at (201.5, 96.7)
- added C3: C_Polarized, Capacitor_THT:CP_Radial_D8.0mm_P3.50mm, F.Cu at (201.3, 112.4)
- added J1: Conn_01x02_Pin, Connector_PinHeader_2.54mm:PinHeader_1x02_P2.54mm_Vertical, F.Cu at (177.0, 93.0)
- added J2: Conn_01x02_Pin, Connector_PinHeader_2.54mm:PinHeader_1x02_P2.54mm_Vertical, F.Cu at (183.1, 101.4)
- added J3: Conn_01x01_Pin, Connector_PinHeader_2.54mm:PinHeader_1x01_P2.54mm_Vertical, F.Cu at (211.2, 96.2)
- added Q1: 2N3904, Package_TO_SOT_THT:TO-92_Inline, F.Cu at (193.9, 103.4)
- added R1: R, Resistor_THT:R_Axial_DIN0207_L6.3mm_D2.5mm_P10.16mm_Horizontal, F.Cu at (189.0, 94.5)
- added R2: R, Resistor_THT:R_Axial_DIN0207_L6.3mm_D2.5mm_P10.16mm_Horizontal, F.Cu at (189.0, 109.5)
- added R3: R, Resistor_THT:R_Axial_DIN0207_L6.3mm_D2.5mm_P10.16mm_Horizontal, F.Cu at (194.0, 119.2)
- added R4: R, Resistor_THT:R_Axial_DIN0207_L6.3mm_D2.5mm_P10.16mm_Horizontal, F.Cu at (193.9, 100.5)
- added R5: R, Resistor_THT:R_Axial_DIN0207_L6.3mm_D2.5mm_P10.16mm_Horizontal, F.Cu at (209.2, 109.4)
- added R6: R, Resistor_THT:R_Axial_DIN0207_L6.3mm_D2.5mm_P10.16mm_Horizontal, F.Cu at (214.7, 109.2)
- added S1: 450301014042, 450301014042:450301014042, F.Cu at (211.9, 104.4)
Routing:
- net +12V: track 0.00 -> 101.1 mm
- net Net-(J3-Pin_1): track 0.00 -> 25.9 mm
- net Net-(Q1-B): track 0.00 -> 15.7 mm
- net Net-(Q1-C): track 0.00 -> 14.8 mm
- net Net-(Q1-E): track 0.00 -> 12.1 mm
- net Net-(R5-Pad1): track 0.00 -> 5.11 mm
- net Net-(R6-Pad1): track 0.00 -> 4.93 mm
- net Net-(J2-Pin_1): track 0.00 -> 4.78 mm
- added copper zone on F.Cu, net GND
Other:
- board size 40 x 25 mm -> 50.7 x 36.2 mm
- board text removed: "Cuadro de Trabajo 4 cm x 3 cm"
