File: grupo-2/Helton/amplificador/amplificador.kicad_pcb (KiCad board)
At the start: 2 copper layers, 40 x 25 mm, 0 parts

Commit message: Actividad Virtual Final
Parts:
- added C1: C_Polarized, Capacitor_THT:CP_Radial_D6.3mm_P2.50mm, F.Cu at (184.4, 91.4)
- added C2: C_Polarized, Capacitor_THT:CP_Radial_D6.3mm_P2.50mm, F.Cu at (185.5, 101.6)
- added C3: C_Polarized, Capacitor_THT:CP_Radial_D6.3mm_P2.50mm, F.Cu at (206.2, 84.5)
- added J1: Conn_01x02_Pin, Connector_PinHeader_2.54mm:PinHeader_1x02_P2.54mm_Vertical, F.Cu at (186.1, 81.2)
- added J2: Conn_01x02_Pin, Connector_PinHeader_2.54mm:PinHeader_1x02_P2.54mm_Vertical, F.Cu at (186.8, 97.0)
- added J3: Conn_01x02_Pin, Connector_PinHeader_2.54mm:PinHeader_1x02_P2.54mm_Vertical, F.Cu at (214.3, 87.0)
- added Q1: 2N3904, Package_TO_SOT_THT:TO-92_Inline, F.Cu at (197.2, 96.7)
- added R1: R, Resistor_THT:R_Axial_DIN0207_L6.3mm_D2.5mm_P10.16mm_Horizontal, F.Cu at (191.9, 81.2)
- added R2: R, Resistor_THT:R_Axial_DIN0207_L6.3mm_D2.5mm_P10.16mm_Horizontal, F.Cu at (191.9, 95.4)
- added R3: R, Resistor_THT:R_Axial_DIN0207_L6.3mm_D2.5mm_P10.16mm_Horizontal, F.Cu at (197.2, 81.2)
- added R4: R, Resistor_THT:R_Axial_DIN0207_L6.3mm_D2.5mm_P10.16mm_Horizontal, F.Cu at (197.3, 99.8)
- added R5: R, Resistor_THT:R_Axial_DIN0207_L6.3mm_D2.5mm_P10.16mm_Horizontal, F.Cu at (205.4, 99.8)
- added R6: R, Resistor_THT:R_Axial_DIN0207_L6.3mm_D2.5mm_P10.16mm_Horizontal, F.Cu at (210.4, 99.8)
- added S1: 450301014042, 450301014042:450301014042, F.Cu at (208.0, 93.6)
Routing:
- net Net-(J3-Pin_2): track 0.00 -> 19.1 mm
- net Net-(Q1-E): track 0.00 -> 15.8 mm
- net Net-(Q1-B): track 0.00 -> 14.3 mm
- net Net-(Q1-C): track 0.00 -> 12.3 mm
- net +12V: track 0.00 -> 11.0 mm
- net Net-(R6-Pad1): track 0.00 -> 6.77 mm
- net Net-(R5-Pad1): track 0.00 -> 6.46 mm
- net SEÑAL: track 0.00 -> 5.67 mm
- added copper zone on F.Cu, net GND
Other:
- board size 40 x 25 mm -> 37.1 x 37.3 mm
- board text removed: "Cuadro de Trabajo 4 cm x 3 cm"
